File: InteractiveElements/Stoplight/Board Design and IO/Esp Controller/Esp Controller.kicad_pcb (KiCad board)
At the start: 2 copper layers, 86.4 x 52.1 mm, 5 parts, among them J1 RJ45, J2 RJ45, J3 RJ45, J4 RJ45, U2 ESP32-DevKitC

Commit message: Update to ESP Pcb
Connections:
- J1 pad 3: unconnected-(J1-Pad3) -> /USBV
- J2 pad 3: unconnected-(J2-Pad3) -> /USBV
- J3 pad 3: unconnected-(J3-Pad3) -> /USBV
- J4 pad 3: unconnected-(J4-Pad3) -> /USBV
- U2 pad 19: unconnected-(U2-5V-Pad19) -> /USBV
Routing:
- net /USBV: track 0.00 -> 119.2 mm

Commit message: modified pcb
Connections:
- J3 pad 6: /Grn1 -> /Grn3
- J4 pad 6: /Grn2 -> /Grn4
- U2 pad 15: unconnected-(U2-MTCK/GPIO13/ADC2_CH4-Pad15) -> /Red3
- U2 pad 20: /Red3 -> unconnected-(U2-SD_CLK/GPIO6-Pad20)
- U2 pad 21: /Blu3 -> unconnected-(U2-SD_DATA0/GPIO7-Pad21)
- U2 pad 22: /Wht3 -> unconnected-(U2-SD_DATA1/GPIO8-Pad22)
- U2 pad 23: /Red2 -> /Grn3
- U2 pad 27: unconnected-(U2-GPIO16-Pad27) -> /Blu3
- U2 pad 28: unconnected-(U2-GPIO17-Pad28) -> /Wht3
- U2 pad 7: unconnected-(U2-32K_XP/GPIO32/ADC1_CH4-Pad7) -> /Red2
- U2 pad 8: unconnected-(U2-32K_XN/GPIO33/ADC1_CH5-Pad8) -> /Wht1
- U2 pad 9: /Wht1 -> /Grn4
Routing:
- net /Grn4: track 0.00 -> 68.2 mm
- net /Grn3: track 0.00 -> 28.9 mm, vias 0 -> 1
- net /Grn1: track 66.1 -> 41.3 mm, vias 1 -> 0
- net /Grn2: track 55.6 -> 32.8 mm
- net /Red3: track 32.8 -> 51.7 mm
- net /Wht3: track 32.9 -> 16.3 mm
- net /Blu3: track 33.3 -> 21.1 mm, vias 0 -> 1
- net /Red2: track 43.8 -> 49.3 mm, vias 0 -> 1
- net /Wht1: track 45.6 -> 50.6 mm
