File: InteractiveElements/Stoplight/Board Design and IO/Esp Controller/Esp Controller.kicad_sch (KiCad schematic)
At the start: 5 parts, among them J1 RJ45, J2 RJ45, J3 RJ45, J4 RJ45, U2 ESP32-DevKitC

Commit message: Update to ESP Pcb
Connections:
- net USBV: now reaches J3.3
- net USBV: now also J1.3, J2.3, J4.3, U2.19 (5V)
Changed lines of the file:
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@@
   (junction (at 222.25 121.92) (diameter 0) (color 0 0 0 0)
   )
+  (wire (pts (xy 207.01 74.93) (xy 228.6 74.93))
+    (stroke (width 0) (type default))
+  )
   (wire (pts (xy 228.6 121.92) (xy 222.25 121.92))
     (stroke (width 0) (type default))
@@
     (stroke (width 0) (type default))
   )
+  (wire (pts (xy 208.28 38.1) (xy 228.6 38.1))
+    (stroke (width 0) (type default))
+  )
   (wire (pts (xy 229.87 45.72) (xy 228.6 45.72))
     (stroke (width 0) (type default))
@@
     (stroke (width 0) (type default))
   )
+  (wire (pts (xy 64.77 24.13) (xy 64.77 20.32))
+    (stroke (width 0) (type default))
+  )
   (wire (pts (xy 217.17 143.51) (xy 217.17 144.78))
     (stroke (width 0) (type default))
@@
     (stroke (width 0) (type default))
   )
+  (wire (pts (xy 208.28 73.66) (xy 207.01 73.66))
+    (stroke (width 0) (type default))
+  )
   (wire (pts (xy 64.77 105.41) (xy 88.9 105.41))
     (stroke (width 0) (type default))
@@
     (stroke (width 0) (type default))
   )
+  (wire (pts (xy 228.6 109.22) (xy 220.98 109.22))
+    (stroke (width 0) (type default))
+  )
   (wire (pts (xy 222.25 119.38) (xy 222.25 121.92))
     (stroke (width 0) (type default))
@@
     (stroke (width 0) (type default))
   )
+  (wire (pts (xy 228.6 140.97) (xy 212.09 140.97))
+    (stroke (width 0) (type default))
+  )
+  (wire (pts (xy 207.01 73.66) (xy 207.01 74.93))
+    (stroke (width 0) (type default))
+  )
   (wire (pts (xy 226.06 85.09) (xy 226.06 82.55))
     (stroke (width 0) (type default))
@@
   )
   (wire (pts (xy 215.9 152.4) (xy 223.52 152.4))
+    (stroke (width 0) (type default))
+  )
+  (wire (pts (xy 64.77 20.32) (xy 76.2 20.32))
     (stroke (width 0) (type default))
   )
@@
     (effects (font (size 1.27 1.27)) (justify left bottom))
   )
+  (label "USBV" (at 76.2 20.32 0) (fields_autoplaced)
+    (effects (font (size 1.27 1.27)) (justify left bottom))
+  )
   (label "Blu1" (at 213.36 40.64 0) (fields_autoplaced)
     (effects (font (size 1.27 1.27)) (justify left bottom))
@@
     (effects (font (size 1.27 1.27)) (justify left bottom))
   )
+  (label "USBV" (at 208.28 73.66 0) (fields_autoplaced)
+    (effects (font (size 1.27 1.27)) (justify left bottom))
+  )
   (label "Blu3" (at 220.98 111.76 0) (fields_autoplaced)
     (effects (font (size 1.27 1.27)) (justify left bottom))
@@
     (effects (font (size 1.27 1.27)) (justify left bottom))
   )
+  (label "USBV" (at 212.09 140.97 0) (fields_autoplaced)
+    (effects (font (size 1.27 1.27)) (justify left bottom))
+  )
   (label "Blu2" (at 105.41 44.45 0) (fields_autoplaced)
     (effects (font (size 1.27 1.27)) (justify left bottom))
@@
     (effects (font (size 1.27 1.27)) (justify left bottom))
   )
+  (label "USBV" (at 208.28 38.1 0) (fields_autoplaced)
+    (effects (font (size 1.27 1.27)) (justify left bottom))
+  )
   (label "Wht2" (at 105.41 49.53 0) (fields_autoplaced)
     (effects (font (size 1.27 1.27)) (justify left bottom))
@@
     (effects (font (size 1.27 1.27)) (justify left bottom))
   )
+  (label "USBV" (at 220.98 109.22 0) (fields_autoplaced)
+    (effects (font (size 1.27 1.27)) (justify left bottom))
+  )

Commit message: modified pcb
Connections:
- net Blu3: now also U2.27 (GPIO16); no longer U2.21 (SD_DATA0/GPIO7)
- net Grn1: no longer J3.6
- net Grn2: no longer J4.6
- net Red2: now also U2.7 (32K_XP/GPIO32/ADC1_CH4); no longer U2.23 (MTDO/GPIO15/ADC2_CH3)
- net Red3: now also U2.15 (MTCK/GPIO13/ADC2_CH4); no longer U2.20 (SD_CLK/GPIO6)
- net Wht1: now also U2.8 (32K_XN/GPIO33/ADC1_CH5); no longer U2.9 (DAC_1/ADC2_CH8/GPIO25)
- net Wht3: now also U2.28 (GPIO17); no longer U2.22 (SD_DATA1/GPIO8)
- new net Grn3: J3.6, U2.23 (MTDO/GPIO15/ADC2_CH3)
- new net Grn4: J4.6, U2.9 (DAC_1/ADC2_CH8/GPIO25)
Changed lines of the file:
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@@
     (stroke (width 0) (type default))
   )
-  (wire (pts (xy 220.98 116.84) (xy 228.6 116.84))
+  (wire (pts (xy 208.28 116.84) (xy 228.6 116.84))
     (stroke (width 0) (type default))
   )
@@
     (stroke (width 0) (type default))
   )
+  (wire (pts (xy 22.86 44.45) (xy 31.75 44.45))
+    (stroke (width 0) (type default))
+  )
   (wire (pts (xy 227.33 147.32) (xy 227.33 146.05))
     (stroke (width 0) (type default))
   )
+  (wire (pts (xy 21.59 49.53) (xy 31.75 49.53))
+    (stroke (width 0) (type default))
+  )
   (wire (pts (xy 213.36 85.09) (xy 226.06 85.09))
     (stroke (width 0) (type default))
@@
     (stroke (width 0) (type default))
   )
+  (wire (pts (xy 21.59 34.29) (xy 31.75 34.29))
+    (stroke (width 0) (type default))
+  )
   (wire (pts (xy 213.36 91.44) (xy 213.36 87.63))
     (stroke (width 0) (type default))
@@
     (stroke (width 0) (type default))
   )
-  (wire (pts (xy 97.79 74.93) (xy 109.22 74.93))
-    (stroke (width 0) (type default))
-  )
   (wire (pts (xy 213.36 35.56) (xy 228.6 35.56))
     (stroke (width 0) (type default))
@@
     (stroke (width 0) (type default))
   )
-  (wire (pts (xy 97.79 77.47) (xy 109.22 77.47))
-    (stroke (width 0) (type default))
-  )
   (wire (pts (xy 227.33 85.09) (xy 228.6 85.09))
     (stroke (width 0) (type default))
   )
-  (wire (pts (xy 97.79 72.39) (xy 109.22 72.39))
-    (stroke (width 0) (type default))
-  )
   (wire (pts (xy 228.6 143.51) (xy 217.17 143.51))
     (stroke (width 0) (type default))
   )
-  (wire (pts (xy 97.79 59.69) (xy 102.87 59.69))
-    (stroke (width 0) (type default))
-  )
   (wire (pts (xy 64.77 24.13) (xy 64.77 20.32))
     (stroke (width 0) (type default))
@@
     (stroke (width 0) (type default))
   )
+  (wire (pts (xy 97.79 90.17) (xy 104.14 90.17))
+    (stroke (width 0) (type default))
+  )
   (wire (pts (xy 228.6 33.02) (xy 213.36 33.02))
     (stroke (width 0) (type default))
@@
     (stroke (width 0) (type default))
   )
+  (wire (pts (xy 97.79 87.63) (xy 104.14 87.63))
+    (stroke (width 0) (type default))
+  )
   (wire (pts (xy 228.6 152.4) (xy 228.6 151.13))
     (stroke (width 0) (type default))
@@
     (stroke (width 0) (type default))
   )
+  (wire (pts (xy 97.79 59.69) (xy 106.68 59.69))
+    (stroke (width 0) (type default))
+  )
   (wire (pts (xy 228.6 149.86) (xy 228.6 148.59))
     (stroke (width 0) (type default))
@@
     (stroke (width 0) (type default))
   )
-  (wire (pts (xy 31.75 49.53) (xy 20.32 49.53))
-    (stroke (width 0) (type default))
-  )
   (wire (pts (xy 214.63 69.85) (xy 228.6 69.85))
     (stroke (width 0) (type default))
@@
   )
   (wire (pts (xy 228.6 40.64) (xy 213.36 40.64))
+    (stroke (width 0) (type default))
+  )
+  (wire (pts (xy 21.59 36.83) (xy 31.75 36.83))
     (stroke (width 0) (type default))
   )
@@
     (effects (font (size 1.27 1.27)) (justify left bottom))
   )
+  (label "Grn3" (at 21.59 49.53 0) (fields_autoplaced)
+    (effects (font (size 1.27 1.27)) (justify left bottom))
+  )
   (label "Red4" (at 217.17 137.16 0) (fields_autoplaced)
     (effects (font (size 1.27 1.27)) (justify left bottom))
   )
-  (label "Grn1" (at 220.98 116.84 0) (fields_autoplaced)
+  (label "Grn3" (at 208.28 116.84 0) (fields_autoplaced)
     (effects (font (size 1.27 1.27)) (justify left bottom))
   )
@@
     (effects (font (size 1.27 1.27)) (justify left bottom))
   )
-  (label "Wht3" (at 109.22 77.47 0) (fields_autoplaced)
+  (label "Wht3" (at 104.14 90.17 0) (fields_autoplaced)
     (effects (font (size 1.27 1.27)) (justify left bottom))
   )
@@
     (effects (font (size 1.27 1.27)) (justify left bottom))
   )
+  (label "Grn2" (at 213.36 85.09 0) (fields_autoplaced)
+    (effects (font (size 1.27 1.27)) (justify left bottom))
+  )
   (label "Blu4" (at 217.17 144.78 0) (fields_autoplaced)
     (effects (font (size 1.27 1.27)) (justify left bottom))
   )
+  (label "Grn4" (at 106.68 59.69 0) (fields_autoplaced)
+    (effects (font (size 1.27 1.27)) (justify left bottom))
+  )
   (label "Wht2" (at 213.36 81.28 0) (fields_autoplaced)
     (effects (font (size 1.27 1.27)) (justify left bottom))
   )
-  (label "Grn2" (at 217.17 149.86 0) (fields_autoplaced)
-    (effects (font (size 1.27 1.27)) (justify left bottom))
-  )
   (label "Yel2" (at 214.63 72.39 0) (fields_autoplaced)
     (effects (font (size 1.27 1.27)) (justify left bottom))
@@
     (effects (font (size 1.27 1.27)) (justify left bottom))
   )
-  (label "Wht1" (at 102.87 59.69 0) (fields_autoplaced)
+  (label "Wht1" (at 21.59 36.83 0) (fields_autoplaced)
     (effects (font (size 1.27 1.27)) (justify left bottom))
   )
@@
     (effects (font (size 1.27 1.27)) (justify left bottom))
   )
-  (label "Red3" (at 109.22 72.39 0) (fields_autoplaced)
-    (effects (font (size 1.27 1.27)) (justify left bottom))
+  (label "Red3" (at 22.86 44.45 180) (fields_autoplaced)
+    (effects (font (size 1.27 1.27)) (justify right bottom))
   )
   (label "Red3" (at 220.98 104.14 0) (fields_autoplaced)
@@
     (effects (font (size 1.27 1.27)) (justify left bottom))
   )
-  (label "Red2" (at 20.32 49.53 0) (fields_autoplaced)
+  (label "Red2" (at 21.59 34.29 0) (fields_autoplaced)
     (effects (font (size 1.27 1.27)) (justify left bottom))
   )
@@
     (effects (font (size 1.27 1.27)) (justify left bottom))
   )
-  (label "Grn2" (at 213.36 85.09 0) (fields_autoplaced)
-    (effects (font (size 1.27 1.27)) (justify left bottom))
-  )
   (label "USBV" (at 220.98 109.22 0) (fields_autoplaced)
     (effects (font (size 1.27 1.27)) (justify left bottom))
@@
     (effects (font (size 1.27 1.27)) (justify left bottom))
   )
-  (label "Blu3" (at 109.22 74.93 0) (fields_autoplaced)
-    (effects (font (size 1.27 1.27)) (justify left bottom))
-  )
+  (label "Grn4" (at 217.17 149.86 0) (fields_autoplaced)
+    (effects (font (size 1.27 1.27)) (justify left bottom))
+  )
+  (label "Blu3" (at 104.14 87.63 0) (fields_autoplaced)
+    (effects (font (size 1.27 1.27)) (justify left bottom))
+  )

Commit message: updated schematic
Connections:
- net USBV: no longer J2.3
Other:
- title: (none) -> Interactive Element Receiver Board
- moved on the sheet: J1, J2, J3, J4, U2
